File: PCB_main/Sofle_Pico.kicad_pcb (KiCad board)
At the start: 2 copper layers, 162.5 x 103 mm, 68 parts, among them J1 Conn_02x08_Top_Bottom, J2 Conn_02x08_Top_Bottom, J3 Conn_02x03, SW1 SW_PUSH, SW10 SW_PUSH, SW11 SW_PUSH, SW12 SW_PUSH, SW13 SW_PUSH, SW14 SW_PUSH, SW15 SW_PUSH, SW16 SW_PUSH, SW17 SW_PUSH, SW18 SW_PUSH, SW2 SW_PUSH, SW20 SW_PUSH, SW21 SW_PUSH, SW22 SW_PUSH, SW23 SW_PUSH, SW24 SW_PUSH, SW27 SW_PUSH, SW28 SW_PUSH, SW29 SW_PUSH, SW3 SW_PUSH, SW30 SW_PUSH, SW37 SW_PUSH, SW38 SW_PUSH, SW39 SW_PUSH, SW4 SW_PUSH, SW40 SW_PUSH, SW41 SW_PUSH, SW5 SW_PUSH, SW6 SW_PUSH, SW7 SW_PUSH, SW8 SW_PUSH, SW9 SW_PUSH, U2 Pico

Commit message: more pcb
Parts:
- moved J2 1.00 mm to (89.5, 38.0)
Routing:
- net row2: track 231.3 -> 246.5 mm, vias 3 -> 4
- net row4: track 235.2 -> 250.2 mm
- net row3: track 231.1 -> 243.0 mm
- net row1: track 222.1 -> 225.1 mm
- net lcol1: track 197.6 -> 195.8 mm
- net row0: track 196.1 -> 195.1 mm
- net lcol6: track 316.6 -> 317.5 mm
- net lcol2: track 257.4 -> 258.1 mm
- net lcol3: track 291.7 -> 292.4 mm
- net lcol4: track 339.2 -> 339.9 mm
- net lcol0: track 169.9 -> 170.7 mm
- net GND: track 61.7 -> 61.2 mm
Other:
- board size 162.5 x 103 mm -> 159.5 x 103 mm

Commit message: thumb cluster connection uses idc
Parts:
- J3: footprint Connector_PinHeader_2.54mm:PinHeader_2x03_P2.54mm_Vertical -> Connector_PinHeader_2.00mm:PinHeader_2x03_P2.00mm_Vertical
- moved J3 25.5 mm to (149.0, 118.4)
- moved D20 13.7 mm to (140.4, 100.5)
- moved D41 12.6 mm to (234.4, 122.0)
Routing:
- net row5: track 104.3 -> 132.7 mm
- net lcol0: track 170.7 -> 197.7 mm
- net row3: track 243.0 -> 262.9 mm
- net lcol3: track 292.4 -> 274.0 mm, vias 2 -> 1
- net lcol2: track 258.1 -> 240.7 mm, vias 2 -> 1
- net lcol4: track 339.9 -> 322.8 mm, vias 2 -> 1
- net lcol1: track 195.8 -> 210.1 mm
- net Net-(D41-A): track 4.09 -> 10.7 mm
- net row4: track 250.2 -> 256.6 mm
- net Net-(D20-A): track 6.02 -> 11.5 mm
Other:
- board text added: "HOWDY!"

Commit message: fix pcb
Parts:
- moved J1 56.4 mm to (82.5, 64.0), turned to 180 degrees
- moved J2 11.4 mm to (80.5, 45.0), turned to 0 degrees
Connections:
- J2 pad 1: row0 -> lcol6
- J2 pad 10: lcol0 -> unconnected-(J2-Pin_10-Pad10)
- J2 pad 11: lcol1 -> row5
- J2 pad 12: lcol2 -> row4
- J2 pad 13: lcol3 -> row3
- J2 pad 14: lcol4 -> row2
- J2 pad 15: lcol5 -> row1
- J2 pad 16: lcol6 -> row0
- J2 pad 2: row1 -> lcol5
- J2 pad 3: row2 -> lcol4
- J2 pad 4: row3 -> lcol3
- J2 pad 5: row4 -> lcol2
- J2 pad 6: row5 -> lcol1
- J2 pad 7: unconnected-(J2-Pin_7-Pad7) -> lcol0
- J2 pad 8: GND -> unconnected-(J2-Pin_8-Pad8)
- J2 pad 9: unconnected-(J2-Pin_9-Pad9) -> GND
- U2 pad 1: row0 -> unconnected-(U2-GPIO0-Pad1)
- U2 pad 2: row1 -> row5
- U2 pad 4: row2 -> row4
- U2 pad 6: row4 -> row2
- U2 pad 7: row5 -> row1
- U2 pad 9: unconnected-(U2-GPIO6-Pad9) -> row0
Routing:
- net lcol6: track 317.5 -> 259.7 mm, vias 1 -> 3
- net lcol5: track 292.8 -> 242.0 mm, vias 1 -> 3
- net lcol4: track 322.8 -> 277.1 mm, vias 1 -> 3
- net lcol0: track 197.7 -> 153.1 mm
- net lcol3: track 274.0 -> 232.9 mm, vias 1 -> 3
- net lcol2: track 240.7 -> 203.4 mm, vias 1 -> 3
- net lcol1: track 210.1 -> 176.0 mm, vias 1 -> 3
- net rcol0: track 64.4 -> 32.6 mm, vias 1 -> 0
- net rcol1: track 64.8 -> 33.1 mm, vias 1 -> 0
- net rcol2: track 57.4 -> 28.2 mm, vias 1 -> 0
- net row5: track 132.7 -> 161.2 mm, vias 2 -> 1
- net rcol3: track 57.7 -> 29.5 mm, vias 1 -> 0
- net rcol4: track 52.7 -> 26.5 mm, vias 1 -> 0
- net rcol5: track 52.6 -> 28.7 mm, vias 1 -> 0
- net row2: track 246.5 -> 226.9 mm, vias 4 -> 2
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Other:
- board size 159.5 x 103 mm -> 166 x 103 mm

Commit message: more pcb work
Connections:
- U2 pad 37: /3V3_EN -> unconnected-(U2-3V3_EN-Pad37)
Routing:
- net row5: track 161.2 -> 160.1 mm
- net lcol3: track 232.9 -> 232.1 mm
