File: PCB_main/Sofle_Pico.kicad_sch (KiCad schematic)
At the start: 68 parts, among them J1 Conn_02x08_Top_Bottom, J2 Conn_02x08_Top_Bottom, J3 Conn_02x03, SW1 SW_PUSH, SW10 SW_PUSH, SW11 SW_PUSH, SW12 SW_PUSH, SW13 SW_PUSH, SW14 SW_PUSH, SW15 SW_PUSH, SW16 SW_PUSH, SW17 SW_PUSH, SW18 SW_PUSH, SW2 SW_PUSH, SW20 SW_PUSH, SW21 SW_PUSH, SW22 SW_PUSH, SW23 SW_PUSH, SW24 SW_PUSH, SW27 SW_PUSH, SW28 SW_PUSH, SW29 SW_PUSH, SW3 SW_PUSH, SW30 SW_PUSH, SW37 SW_PUSH, SW38 SW_PUSH, SW39 SW_PUSH, SW4 SW_PUSH, SW40 SW_PUSH, SW41 SW_PUSH, SW5 SW_PUSH, SW6 SW_PUSH, SW7 SW_PUSH, SW8 SW_PUSH, SW9 SW_PUSH, U2 Pico

Commit message: more pcb work
Connections:
- net 3V3_EN: no longer names the net of U2.37 (3V3_EN)
- no-connect marks 5 -> 16
Changed lines of the file:
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@@
+	)
+	(no_connect
+		(at 81.28 41.91)
 	)
 	(no_connect
@@
 	)
 	(no_connect
+		(at 129.54 44.45)
+	)
+	(no_connect
+		(at 199.39 81.28)
+	)
+	(no_connect
 		(at 234.95 93.98)
 	)
@@
 	)
 	(no_connect
+		(at 234.95 104.14)
+	)
+	(no_connect
+		(at 234.95 96.52)
+	)
+	(no_connect
+		(at 234.95 101.6)
+	)
+	(no_connect
+		(at 129.54 41.91)
+	)
+	(no_connect
+		(at 234.95 88.9)
+	)
+	(no_connect
+		(at 199.39 106.68)
+	)
+	(no_connect
+		(at 199.39 109.22)
+	)
+	(no_connect
 		(at 219.71 134.62)
 	)
@@
 		(at 234.95 106.68)
 	)
+	(no_connect
+		(at 81.28 44.45)
+	)
 	(wire
 		(pts
@@
 	(wire
 		(pts
-			(xy 234.95 88.9) (xy 243.205 88.9)
-		)
-		(stroke
-			(width 0)
-			(type default)
-		)
-	)
-	(wire
-		(pts
 			(xy 152.4 124.46) (xy 152.4 140.97)
 		)
@@
 		)
 	)
-	(label "3V3_EN"
-		(at 236.22 88.9 0)
-		(effects
-			(font
-				(size 1.27 1.27)
-			)
-			(justify left bottom)
-		)
-	)
